File: hw/_saved_NotACamera.sch (KiCad schematic (older format))
At the start: 8 parts, among them U1 7555

Commit message: Finished initial layout
Parts:
- P1: renamed from P?; value CONN_02X02 -> SAO; footprint (none) -> Pin_Headers:Pin_Header_Straight_2x02
Changed lines of the file:
@@
 VCC
 $Comp
-L CONN_02X02 P?
+L CONN_02X02 P1
 U 1 1 5B458FE1
 P 3750 2950
-F 0 "P?" H 3750 3100 50  0000 C CNN
-F 1 "CONN_02X02" H 3750 2800 50  0000 C CNN
-F 2 "" H 3750 1750 50  0000 C CNN
+F 0 "P1" H 3750 3100 50  0000 C CNN
+F 1 "SAO" H 3750 2800 50  0000 C CNN
+F 2 "Pin_Headers:Pin_Header_Straight_2x02" H 3750 1750 50  0001 C CNN
 F 3 "" H 3750 1750 50  0000 C CNN
 	1    3750 2950
