File: hw/NotACamera.sch (KiCad schematic (older format))
At the start: 8 parts, among them U1 7555

Commit message: Finished initial layout
Parts:
- removed BT1: CR2032, Firefly:S8211R, symbol Battery
- added P1: SAO, symbol CONN_02X02
Connections:
- wire segments 21 -> 23
Changed lines of the file:
@@
 LIBS:valves
 LIBS:7555
-LIBS:DigitalFirefly-cache
 EELAYER 25 0
 EELAYER END
@@
 	0    1    1    0
 $EndComp
-$Comp
-L Battery BT1
-U 1 1 5B2D7800
-P 3400 2975
-F 0 "BT1" H 3500 3025 50  0000 L CNN
-F 1 "CR2032" H 3500 2925 50  0000 L CNN
-F 2 "Firefly:S8211R" V 3400 3015 50  0001 C CNN
-F 3 "" V 3400 3015 50  0000 C CNN
-	1    3400 2975
-	1    0    0    -1
-$EndComp
 Wire Wire Line
-	3400 2825 3400 1775
+	3400 1775 3400 2900
 Wire Wire Line
 	3400 1775 7500 1775
@@
 	5650 1775 5650 2075
 Wire Wire Line
-	3400 3125 3400 4275
+	3400 3000 3400 4275
 Wire Wire Line
 	3400 4275 7500 4275
@@
 Text Label 5125 1775 0    60   ~ 0
 VCC
+$Comp
+L CONN_02X02 P1
+U 1 1 5B458FE1
+P 3750 2950
+F 0 "P1" H 3750 3100 50  0000 C CNN
+F 1 "SAO" H 3750 2800 50  0000 C CNN
+F 2 "" H 3750 1750 50  0000 C CNN
+F 3 "" H 3750 1750 50  0000 C CNN
+	1    3750 2950
+	1    0    0    -1
+$EndComp
+Wire Wire Line
+	3400 2900 3500 2900
+Wire Wire Line
+	3500 3000 3400 3000
 $EndSCHEMATC

Commit message: Changed schematic for new connections, values and footprint associations
Parts:
- C1, C2: footprint Capacitors_SMD:C_1210 -> Resistors_SMD:R_0805_HandSoldering; MPN (none) -> MPN
- D1: footprint LEDs:LED_0805 -> Resistors_SMD:R_0805_HandSoldering; symbol LED -> LED-RESCUE-NotACamera; MPN (none) -> MPN
- P1: footprint (none) -> Pin_Headers:Pin_Header_Straight_2x02
- R1: value 1K8 -> 100; footprint Resistors_SMD:R_0805 -> Resistors_SMD:R_0805_HandSoldering; MPN (none) -> MPN
- R2: value 220K -> 100; footprint Resistors_SMD:R_0805 -> Resistors_SMD:R_0805_HandSoldering; MPN (none) -> MPN
- R3: value 1K8 -> 68K; footprint Resistors_SMD:R_0805 -> Resistors_SMD:R_0805_HandSoldering; MPN (none) -> MPN
Connections:
- net GND: now also D1.1 (K)
- net VCC: now also R2.1; no longer D1.2 (A)
- net at U1.7 (Discharge): now also R2.2, R3.1; no longer R2.1
- net at C1.1, R3.2, U1.6 (Threshold): now also U1.2 (~Trigger)
- net at R1.2: now also D1.2 (A); no longer D1.1 (K)
Other:
- moved on the sheet: D1, R2, R3
Changed lines of the file:
@@
 EESchema Schematic File Version 2
+LIBS:NotACamera-rescue
 LIBS:power
 LIBS:device
@@
 LIBS:valves
 LIBS:7555
+LIBS:NotACamera-cache
 EELAYER 25 0
 EELAYER END
@@
 L R R2
 U 1 1 5B2D7368
-P 6625 2775
-F 0 "R2" V 6705 2775 50  0000 C CNN
-F 1 "220K" V 6625 2775 50  0000 C CNN
-F 2 "Resistors_SMD:R_0805" V 6555 2775 50  0001 C CNN
-F 3 "" H 6625 2775 50  0000 C CNN
-	1    6625 2775
+P 6625 2275
+F 0 "R2" V 6705 2275 50  0000 C CNN
+F 1 "100" V 6625 2275 50  0000 C CNN
+F 2 "Resistors_SMD:R_0805_HandSoldering" V 6555 2275 50  0001 C CNN
+F 3 "" H 6625 2275 50  0000 C CNN
+F 4 "MPN" H 6625 2275 60  0001 C CNN "MPN"
+	1    6625 2275
 	1    0    0    -1
 $EndComp
@@
 L R R3
 U 1 1 5B2D7385
-P 6625 3225
-F 0 "R3" V 6705 3225 50  0000 C CNN
-F 1 "1K8" V 6625 3225 50  0000 C CNN
-F 2 "Resistors_SMD:R_0805" V 6555 3225 50  0001 C CNN
-F 3 "" H 6625 3225 50  0000 C CNN
-	1    6625 3225
+P 6625 2775
+F 0 "R3" V 6705 2775 50  0000 C CNN
+F 1 "68K" V 6625 2775 50  0000 C CNN
+F 2 "Resistors_SMD:R_0805_HandSoldering" V 6555 2775 50  0001 C CNN
+F 3 "" H 6625 2775 50  0000 C CNN
+F 4 "MPN" H 6625 2775 60  0001 C CNN "MPN"
+	1    6625 2775
 	1    0    0    -1
 $EndComp
@@
 F 0 "C1" H 6650 3850 50  0000 L CNN
 F 1 "10U" H 6650 3650 50  0000 L CNN
-F 2 "Capacitors_SMD:C_1210" H 6663 3600 50  0001 C CNN
+F 2 "Resistors_SMD:R_0805_HandSoldering" H 6663 3600 50  0001 C CNN
 F 3 "" H 6625 3750 50  0000 C CNN
+F 4 "MPN" H 6625 3750 60  0001 C CNN "MPN"
 	1    6625 3750
 	1    0    0    -1
@@
 F 0 "C2" H 7525 3450 50  0000 L CNN
 F 1 "10U" H 7525 3250 50  0000 L CNN
-F 2 "Capacitors_SMD:C_1210" H 7538 3200 50  0001 C CNN
+F 2 "Resistors_SMD:R_0805_HandSoldering" H 7538 3200 50  0001 C CNN
 F 3 "" H 7500 3350 50  0000 C CNN
+F 4 "MPN" H 7500 3350 60  0001 C CNN "MPN"
 	1    7500 3350
 	1    0    0    -1
 $EndComp
 $Comp
-L LED D1
+L LED-RESCUE-NotACamera D1
 U 1 1 5B2D76A7
-P 4250 2400
-F 0 "D1" H 4250 2500 50  0000 C CNN
-F 1 "GREEN LED" H 4250 2300 50  0000 C CNN
-F 2 "LEDs:LED_0805" H 4250 2400 50  0001 C CNN
-F 3 "" H 4250 2400 50  0000 C CNN
-	1    4250 2400
+P 4250 3425
+F 0 "D1" H 4250 3525 50  0000 C CNN
+F 1 "GREEN LED" H 4250 3325 50  0000 C CNN
+F 2 "Resistors_SMD:R_0805_HandSoldering" H 4250 3425 50  0001 C CNN
+F 3 "" H 4250 3425 50  0000 C CNN
+F 4 "MPN" H 4250 3425 60  0001 C CNN "MPN"
+	1    4250 3425
 	0    -1   -1   0
 $EndComp
@@
 P 4525 2975
 F 0 "R1" V 4605 2975 50  0000 C CNN
-F 1 "1K8" V 4525 2975 50  0000 C CNN
-F 2 "Resistors_SMD:R_0805" V 4455 2975 50  0001 C CNN
+F 1 "100" V 4525 2975 50  0000 C CNN
+F 2 "Resistors_SMD:R_0805_HandSoldering" V 4455 2975 50  0001 C CNN
 F 3 "" H 4525 2975 50  0000 C CNN
+F 4 "MPN" H 4525 2975 60  0001 C CNN "MPN"
 	1    4525 2975
 	0    1    1    0
@@
 	5650 4275 5650 3925
 Wire Wire Line
-	4250 2200 4250 1775
-Connection ~ 4250 1775
-Wire Wire Line
-	4250 2600 4250 2975
-Wire Wire Line
 	4250 2975 4375 2975
 Wire Wire Line
@@
 	6450 2575 6625 2575
 Wire Wire Line
-	6625 2575 6625 2625
-Wire Wire Line
-	6625 2925 6625 3075
+	6625 2425 6625 2625
+Wire Wire Line
+	6625 2925 6625 3600
 Wire Wire Line
 	6450 2975 6625 2975
@@
 Wire Wire Line
 	6450 3475 6625 3475
-Wire Wire Line
-	6625 3375 6625 3600
 Connection ~ 6625 3475
 Wire Wire Line
@@
 F 0 "P1" H 3750 3100 50  0000 C CNN
 F 1 "SAO" H 3750 2800 50  0000 C CNN
-F 2 "" H 3750 1750 50  0000 C CNN
+F 2 "Pin_Headers:Pin_Header_Straight_2x02" H 3750 1750 50  0001 C CNN
 F 3 "" H 3750 1750 50  0000 C CNN
 	1    3750 2950
@@
 Wire Wire Line
 	3500 3000 3400 3000
+Wire Wire Line
+	4250 2975 4250 3225
+Wire Wire Line
+	4250 3625 4250 4275
+Connection ~ 4250 4275
+Wire Wire Line
+	6625 2125 6625 1775
+Connection ~ 6625 1775
+Connection ~ 6625 2575
 $EndSCHEMATC
